Commit message: converted joints to continuous

File: tribot_description/urdf/tribot.urdf (robot description, URDF)
Before this commit: robot tribot, 10 links, 9 joints
Joints:
- joint c_body_to_l_triplet: limit lower=-3.14159 upper=3.14159 effort=0 velocity=0 -> (none); type revolute -> continuous
- joint c_body_to_r_triplet: limit lower=-3.14159 upper=3.14159 effort=0 velocity=0 -> (none); type revolute -> continuous
- joint l_triplet_to_l_wheel_1: limit lower=-3.14159 upper=3.14159 effort=0 velocity=0 -> (none); type revolute -> continuous
- joint l_triplet_to_l_wheel_2: limit lower=-3.14159 upper=3.14159 effort=0 velocity=0 -> (none); type revolute -> continuous
- joint l_triplet_to_l_wheel_3: limit lower=-3.14159 upper=3.14159 effort=0 velocity=0 -> (none); type revolute -> continuous
- joint r_triplet_to_r_wheel_1: limit lower=-3.14159 upper=3.14159 effort=0 velocity=0 -> (none); type revolute -> continuous
- joint r_triplet_to_r_wheel_2: limit lower=-3.14159 upper=3.14159 effort=0 velocity=0 -> (none); type revolute -> continuous
- joint r_triplet_to_r_wheel_3: limit lower=-3.14159 upper=3.14159 effort=0 velocity=0 -> (none); type revolute -> continuous
